File: Circuits/MotherPCB/PT.kicad_sch (KiCad schematic)
At the start: 0 parts

Commit message: cleaned up the lib folder of microcontroller code
Parts:
- added J2: Raspberry_Pi_2_3, symbol Connector:Raspberry_Pi_2_3
Connections:
- new net: J2.1 (3V3), J2.17 (3V3)
- new net: J2.14 (GND), J2.20 (GND), J2.25 (GND), J2.30 (GND), J2.34 (GND), J2.39 (GND), J2.6 (GND), J2.9 (GND)
- new net: J2.2 (5V), J2.4 (5V)
- new net CS: J2.15 (GPIO22)
- new net DIN: J2.21 (MISO0/GPIO9)
- new net DO: J2.19 (MOSI0/GPIO10)
- new net DRDY: J2.11 (GPIO17)
- new net SCK: J2.23 (SCLK0/GPIO11)
