File: Circuits/MotherPCB/LoadCell.kicad_sch (KiCad schematic)
At the start: 0 parts

Commit message: Done for the night
Finished up thermocouple differential communication and every other module apart from PTs and Oil Injector.

Good night.
oh wait
It's 4:00 am.
Good morning
Parts:
- added C2: 0.1uF, PCM_SparkFun-Capacitor:C_0402_1005Metric, symbol PCM_SparkFun-Capacitor:0.1uF_0402_16V_10%
- added J8: HX711, Connector_PinHeader_2.54mm:PinHeader_1x04_P2.54mm_Vertical, symbol PCM_SL_Pin_Headers:PINHD_1x4_Male
Connections:
- new net 3V3: C2.2, J8.1
- new net GND: C2.1, J8.4
- new net MISO: J8.3
- new net SCK: J8.2
Other:
- note added: "DT"
- note added: "GND"
- note added: "SCK"
- note added: "VCC"

Commit message: pcb completed with a clean DRC
first one it is let us pray it works
Parts:
- C2: footprint PCM_SparkFun-Capacitor:C_0402_1005Metric -> Capacitor_THT:C_Disc_D5.0mm_W2.5mm_P5.00mm
Changed lines of the file:
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@@
 			)
 		)
-		(property "Footprint" "PCM_SparkFun-Capacitor:C_0402_1005Metric"
+		(property "Footprint" "Capacitor_THT:C_Disc_D5.0mm_W2.5mm_P5.00mm"
 			(at 115.57 93.98 0)
 			(effects
