File: Circuits/MotherPCB/Oiljector.kicad_sch (KiCad schematic)
At the start: 0 parts

Commit message: Added footprint for ATTiny85 module, added schematic for oil injector circuit
Parts:
- added I: ~, Additional_Components:Digispark_ATTiny85_Headers, symbol Additional_Components:Digispark_ATTiny85
- added J19: Conn_01x06_Socket, symbol Connector:Conn_01x06_Socket
Connections:
- new net 5V: J19.1 (Pin_1)
- new net GND: J19.6 (Pin_6)
Other:
- note added: "GND"
- note added: "Sockets for ULN2003A stepper driver modules"
- note added: "Vin"
- company: (none) -> Project Arka
- title: (none) -> Oiling Stepper Control

Commit message: Added Teensy and some labels to the schematic
Parts:
- renumbered I to I2
Changed lines of the file:
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@@
 		(dnp no)
 		(fields_autoplaced yes)
-		(property "Reference" "I"
+		(property "Reference" "I?"
 			(at 137.16 93.98 0)
 			(effects
@@
 					(unit 1)
 				)
+				(path "/ea485091-218e-4ddf-97d6-ebaac999a2f0/c0496eb1-5cec-499b-a2b9-c70299f0e30e"
+					(reference "I?")
+					(unit 1)
+				)

Commit message: Schematic Finished
Parts:
- J19: footprint (none) -> Connector_PinHeader_2.54mm:PinHeader_1x06_P2.54mm_Vertical
Changed lines of the file:
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@@
 			)
 		)
-		(property "Footprint" ""
+		(property "Footprint" "Connector_PinHeader_2.54mm:PinHeader_1x06_P2.54mm_Vertical"
 			(at 88.9 95.25 0)
 			(effects

Commit message: Fixed some broken footprints
Parts:
- renumbered I2 to I1
Changed lines of the file:
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@@
 		(dnp no)
 		(fields_autoplaced yes)
-		(property "Reference" "I?"
+		(property "Reference" "I1"
 			(at 137.16 93.98 0)
 			(effects
@@
 				)
 				(path "/ea485091-218e-4ddf-97d6-ebaac999a2f0/c0496eb1-5cec-499b-a2b9-c70299f0e30e"
-					(reference "I?")
+					(reference "I1")
 					(unit 1)
 				)

Commit message: pcb completed with a clean DRC
first one it is let us pray it works
Connections:
- net 5V: now also I1.8 (5V)
- net GND: now also I1.7 (GND)
- net TGR: now also I1.0 (P0/MOSI)
- net at J19.2 (Pin_2): now also I1.1 (P1/MISO)
- net at J19.3 (Pin_3): now also I1.2 (P2/SCK)
- net at J19.4 (Pin_4): now also I1.3 (P3)
- net at J19.5 (Pin_5): now also I1.4 (P4)
- no-connect marks 0 -> 2
Changed lines of the file:
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@@
 	)
 	(junction
-		(at 158.75 87.63)
+		(at 142.24 82.55)
 		(diameter 0)
-		(color 0 0 0 1)
-	)
-	(junction
-		(at 138.43 82.55)
-		(diameter 0)
-		(color 255 0 0 1)
-	)
-	(wire
-		(pts
-			(xy 93.98 82.55) (xy 138.43 82.55)
+		(color 0 0 0 0)
+	)
+	(no_connect
+		(at 139.7 86.36)
+	)
+	(no_connect
+		(at 132.08 99.06)
+	)
+	(wire
+		(pts
+			(xy 93.98 93.98) (xy 93.98 92.71)
+		)
+		(stroke
+			(width 0)
+			(type default)
+		)
+	)
+	(wire
+		(pts
+			(xy 132.08 93.98) (xy 93.98 93.98)
+		)
+		(stroke
+			(width 0)
+			(type default)
+		)
+	)
+	(wire
+		(pts
+			(xy 132.08 96.52) (xy 93.98 96.52)
+		)
+		(stroke
+			(width 0)
+			(type default)
+		)
+	)
+	(wire
+		(pts
+			(xy 96.52 97.79) (xy 96.52 100.33)
+		)
+		(stroke
+			(width 0)
+			(type default)
+		)
+	)
+	(wire
+		(pts
+			(xy 140.97 85.09) (xy 158.75 85.09)
+		)
+		(stroke
+			(width 0)
+			(type default)
+		)
+	)
+	(wire
+		(pts
+			(xy 93.98 96.52) (xy 93.98 97.79)
+		)
+		(stroke
+			(width 0)
+			(type default)
+		)
+	)
+	(wire
+		(pts
+			(xy 93.98 95.25) (xy 132.08 95.25)
+		)
+		(stroke
+			(width 0)
+			(type default)
+		)
+	)
+	(wire
+		(pts
+			(xy 93.98 82.55) (xy 142.24 82.55)
 		)
 		(stroke
@@
 	(wire
 		(pts
-			(xy 93.98 93.98) (xy 93.98 92.71)
-		)
-		(stroke
-			(width 0)
-			(type default)
-		)
-	)
-	(wire
-		(pts
-			(xy 132.08 93.98) (xy 93.98 93.98)
-		)
-		(stroke
-			(width 0)
-			(type default)
-		)
-	)
-	(wire
-		(pts
-			(xy 132.08 96.52) (xy 93.98 96.52)
-		)
-		(stroke
-			(width 0)
-			(type default)
-		)
-	)
-	(wire
-		(pts
-			(xy 139.7 87.63) (xy 158.75 87.63)
+			(xy 93.98 90.17) (xy 93.98 82.55)
+		)
+		(stroke
+			(width 0)
+			(type default)
+			(color 255 0 0 1)
+		)
+	)
+	(wire
+		(pts
+			(xy 132.08 92.71) (xy 129.54 92.71)
+		)
+		(stroke
+			(width 0)
+			(type default)
+		)
+	)
+	(wire
+		(pts
+			(xy 158.75 85.09) (xy 158.75 102.87)
 		)
 		(stroke
@@
 	(wire
 		(pts
-			(xy 96.52 97.79) (xy 96.52 100.33)
-		)
-		(stroke
-			(width 0)
-			(type default)
-		)
-	)
-	(wire
-		(pts
-			(xy 93.98 96.52) (xy 93.98 97.79)
-		)
-		(stroke
-			(width 0)
-			(type default)
-		)
-	)
-	(wire
-		(pts
-			(xy 93.98 95.25) (xy 132.08 95.25)
-		)
-		(stroke
-			(width 0)
-			(type default)
-		)
-	)
-	(wire
-		(pts
-			(xy 139.7 88.9) (xy 139.7 87.63)
-		)
-		(stroke
-			(width 0)
-			(type default)
-		)
-	)
-	(wire
-		(pts
-			(xy 138.43 82.55) (xy 158.75 82.55)
+			(xy 142.24 82.55) (xy 142.24 86.36)
+		)
+		(stroke
+			(width 0)
+			(type default)
+		)
+	)
+	(wire
+		(pts
+			(xy 132.08 97.79) (xy 96.52 97.79)
+		)
+		(stroke
+			(width 0)
+			(type default)
+		)
+	)
+	(wire
+		(pts
+			(xy 96.52 100.33) (xy 93.98 100.33)
+		)
+		(stroke
+			(width 0)
+			(type default)
+		)
+	)
+	(wire
+		(pts
+			(xy 129.54 92.71) (xy 129.54 80.01)
+		)
+		(stroke
+			(width 0)
+			(type default)
+		)
+	)
+	(wire
+		(pts
+			(xy 129.54 80.01) (xy 158.75 80.01)
+		)
+		(stroke
+			(width 0)
+			(type default)
+		)
+	)
+	(wire
+		(pts
+			(xy 93.98 102.87) (xy 158.75 102.87)
+		)
+		(stroke
+			(width 0)
+			(type default)
+			(color 0 0 0 1)
+		)
+	)
+	(wire
+		(pts
+			(xy 140.97 86.36) (xy 140.97 85.09)
+		)
+		(stroke
+			(width 0)
+			(type default)
+		)
+	)
+	(wire
+		(pts
+			(xy 142.24 82.55) (xy 158.75 82.55)
 		)
 		(stroke
@@
 			(type default)
 			(color 255 0 0 1)
-		)
-	)
-	(wire
-		(pts
-			(xy 93.98 90.17) (xy 93.98 82.55)
-		)
-		(stroke
-			(width 0)
-			(type default)
-			(color 255 0 0 1)
-		)
-	)
-	(wire
-		(pts
-			(xy 132.08 92.71) (xy 129.54 92.71)
-		)
-		(stroke
-			(width 0)
-			(type default)
-		)
-	)
-	(wire
-		(pts
-			(xy 138.43 82.55) (xy 138.43 88.9)
-		)
-		(stroke
-			(width 0)
-			(type default)
-			(color 255 0 0 1)
-		)
-	)
-	(wire
-		(pts
-			(xy 158.75 87.63) (xy 158.75 85.09)
-		)
-		(stroke
-			(width 0)
-			(type default)
-			(color 0 0 0 1)
-		)
-	)
-	(wire
-		(pts
-			(xy 132.08 97.79) (xy 96.52 97.79)
-		)
-		(stroke
-			(width 0)
-			(type default)
-		)
-	)
-	(wire
-		(pts
-			(xy 96.52 100.33) (xy 93.98 100.33)
-		)
-		(stroke
-			(width 0)
-			(type default)
-		)
-	)
-	(wire
-		(pts
-			(xy 129.54 92.71) (xy 129.54 80.01)
-		)
-		(stroke
-			(width 0)
-			(type default)
-		)
-	)
-	(wire
-		(pts
-			(xy 129.54 80.01) (xy 158.75 80.01)
-		)
-		(stroke
-			(width 0)
-			(type default)
-		)
-	)
-	(wire
-		(pts
-			(xy 158.75 102.87) (xy 158.75 87.63)
-		)
-		(stroke
-			(width 0)
-			(type default)
-			(color 0 0 0 1)
-		)
-	)
-	(wire
-		(pts
-			(xy 93.98 102.87) (xy 158.75 102.87)
-		)
-		(stroke
-			(width 0)
-			(type default)
-			(color 0 0 0 1)
 		)
 	)
@@
 	(symbol
 		(lib_id "Additional_Components:Digispark_ATTiny85")
-		(at 137.16 93.98 0)
+		(at 138.43 93.98 0)
 		(unit 1)
 		(exclude_from_sim no)
@@
 		(fields_autoplaced yes)
 		(property "Reference" "I1"
-			(at 137.16 93.98 0)
+			(at 138.43 93.98 0)
 			(effects
 				(font
@@
 		)
 		(property "Value" "~"
-			(at 137.16 86.36 0)
-			(effects
-				(font
-					(size 1.27 1.27)
-				)
+			(at 138.43 86.36 0)
+			(effects
+				(font
+					(size 1.27 1.27)
+				)
+				(hide yes)
 			)
 		)
 		(property "Footprint" "Additional_Components:Digispark_ATTiny85_Headers"
-			(at 137.16 93.98 0)
+			(at 138.43 93.98 0)
 			(effects
 				(font
@@
 		)
 		(property "Datasheet" "https://robu.in/wp-content/uploads/2017/06/ATTINY85-USB-Development-Board-Dimensional-Drawing-ROBU.IN_.pdf"
-			(at 137.16 93.98 0)
+			(at 138.43 93.98 0)
 			(effects
 				(font
@@
 		)
 		(property "Description" "Headers for the ATTiny85 dev board by Digispark"
-			(at 137.16 93.98 0)
+			(at 138.43 93.98 0)
 			(effects
 				(font
@@
 		(pin "1"
 		)
-		(pin ""
-		)
-		(pin ""
-		)
-		(pin ""
+		(pin "8"
+		)
+		(pin "7"
+		)
+		(pin "6"
 		)
 		(pin "5"
