File: Circuits/MotherPCB/Tachometer.kicad_sch (KiCad schematic)
At the start: 4 parts, among them J4 Conn_01x03_Pin, Q1 BSS138W

Commit message: pcb completed with a clean DRC
first one it is let us pray it works
Parts:
- removed C19: 0.1uF, PCM_SparkFun-Capacitor:C_0402_1005Metric, symbol PCM_SparkFun-Capacitor:0.1uF_0402_16V_10%
- removed Q1: BSS138W, PCM_Package_TO_SOT_SMD_AKL:SOT-323_SC-70, symbol PCM_Transistor_MOSFET_AKL:BSS138W
- removed R9: 10k, PCM_SparkFun-Resistor:R_0603_1608Metric, symbol PCM_SparkFun-Resistor:10k_0603
- added R20, R21, R9: 10k, Resistor_THT:R_Axial_DIN0207_L6.3mm_D2.5mm_P7.62mm_Horizontal, symbol Device:R
Connections:
- net 5V: now also J4.2 (Pin_2); no longer J4.1 (Pin_1)
- net GND: now also J4.3 (Pin_3), R9.2; no longer J4.2 (Pin_2)
- new net: J4.1 (Pin_1), R21.1
- new net: R20.2, R9.1
- new net SIG: R20.1, R21.2
