File: Circuits/MotherPCB/Thermocouple.kicad_sch (KiCad schematic)
At the start: 0 parts

Commit message: Done for the night
Finished up thermocouple differential communication and every other module apart from PTs and Oil Injector.

Good night.
oh wait
It's 4:00 am.
Good morning
Parts:
- added C10, C9: 0.1uF, Capacitor_SMD:C_0201_0603Metric, symbol PCM_SparkFun-Capacitor:C_Small
- added J11: USB3_A, symbol Connector:USB3_A
- added R4: 120, Resistor_SMD:R_0201_0603Metric, symbol Device:R
- added U8, U9: MAX3485, Package_SO:SOIC-8_3.9x4.9mm_P1.27mm, symbol Interface_UART:MAX3485
Connections:
- new net: J11.8 (SSTX-), R4.1, U9.7 (B)
- new net: J11.9 (SSTX+), R4.2, U9.6 (A)
- new net: J11.5 (SSRX-), U8.7 (B)
- new net: J11.6 (SSRX+), U8.6 (A)
- new net 3.3V: C10.2, C9.2, J11.1 (VBUS), U8.2 (~{RE}), U8.3 (DE), U8.8 (VCC), U9.8 (VCC)
- new net CS: J11.2 (D-), J11.3 (D+)
- new net GND: C10.1, C9.1, J11.4 (GND), U8.5 (GND), U9.2 (~{RE}), U9.3 (DE), U9.5 (GND)
- new net MISO: U9.4 (DI)
- new net SCK: U8.4 (DI)
Other:
- note added: "CLOCK"
- note added: "MISO"

Commit message: Fixed some broken footprints
Parts:
- J18: renamed from J11; footprint (none) -> Additional_Components:SAMTEC_USB3-A-S-F-TH
- renumbered C9 to C20, C10 to C21, R4 to R10, U8 to U19, U9 to U21
Changed lines of the file:
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@@
 		(on_board yes)
 		(dnp no)
-		(property "Reference" "R?"
+		(property "Reference" "R10"
 			(at 110.49 143.5099 0)
 			(effects
@@
 				)
 				(path "/ea485091-218e-4ddf-97d6-ebaac999a2f0/da95a8c2-1e5d-4053-8fb4-7b6063b75ac8"
-					(reference "R?")
+					(reference "R10")
 					(unit 1)
 				)
@@
 		(dnp no)
 		(fields_autoplaced yes)
-		(property "Reference" "C?"
+		(property "Reference" "C21"
 			(at 156.21 149.8662 0)
 			(effects
@@
 				)
 				(path "/ea485091-218e-4ddf-97d6-ebaac999a2f0/da95a8c2-1e5d-4053-8fb4-7b6063b75ac8"
-					(reference "C?")
+					(reference "C21")
 					(unit 1)
 				)
@@
 		(dnp no)
 		(fields_autoplaced yes)
-		(property "Reference" "C?"
+		(property "Reference" "C20"
 			(at 156.21 102.8762 0)
 			(effects
@@
 				)
 				(path "/ea485091-218e-4ddf-97d6-ebaac999a2f0/da95a8c2-1e5d-4053-8fb4-7b6063b75ac8"
-					(reference "C?")
+					(reference "C20")
 					(unit 1)
 				)
@@
 		(dnp no)
 		(fields_autoplaced yes)
-		(property "Reference" "J?"
+		(property "Reference" "J18"
 			(at 77.47 91.44 0)
 			(effects
@@
 			)
 		)
-		(property "Footprint" ""
+		(property "Footprint" "Additional_Components:SAMTEC_USB3-A-S-F-TH"
 			(at 81.28 107.95 0)
 			(effects
@@
 				)
 				(path "/ea485091-218e-4ddf-97d6-ebaac999a2f0/da95a8c2-1e5d-4053-8fb4-7b6063b75ac8"
-					(reference "J?")
+					(reference "J18")
 					(unit 1)
 				)
@@
 		(dnp no)
 		(fields_autoplaced yes)
-		(property "Reference" "U?"
+		(property "Reference" "U21"
 			(at 142.8181 120.65 0)
 			(effects
@@
 				)
 				(path "/ea485091-218e-4ddf-97d6-ebaac999a2f0/da95a8c2-1e5d-4053-8fb4-7b6063b75ac8"
-					(reference "U?")
+					(reference "U21")
 					(unit 1)
 				)
@@
 		(dnp no)
 		(fields_autoplaced yes)
-		(property "Reference" "U?"
+		(property "Reference" "U19"
 			(at 142.8181 71.12 0)
 			(effects
@@
 				)
 				(path "/ea485091-218e-4ddf-97d6-ebaac999a2f0/da95a8c2-1e5d-4053-8fb4-7b6063b75ac8"
-					(reference "U?")
-					(unit 1)
-				)
+					(reference "U19")
+					(unit 1)
+				)

Commit message: pcb completed with a clean DRC
first one it is let us pray it works
Parts:
- removed C20: 0.1uF, Capacitor_SMD:C_0201_0603Metric, symbol PCM_SparkFun-Capacitor:C_Small
- added C3: 0.1uF, Capacitor_THT:C_Disc_D5.0mm_W2.5mm_P5.00mm, symbol PCM_SparkFun-Capacitor:C_Small
- C21: footprint Capacitor_SMD:C_0201_0603Metric -> Capacitor_THT:C_Disc_D5.0mm_W2.5mm_P5.00mm
- R10: footprint Resistor_SMD:R_0201_0603Metric -> Resistor_THT:R_Axial_DIN0207_L6.3mm_D2.5mm_P7.62mm_Horizontal
Connections:
- net 3.3V: now also C3.2
- net GND: now also C3.1
- net MISO: now also U21.1 (RO); no longer U21.4 (DI)
- no-connect marks 0 -> 4
Changed lines of the file:
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@@
 		(color 0 0 0 0)
 	)
+	(no_connect
+		(at 74.93 128.27)
+	)
+	(no_connect
+		(at 149.86 93.98)
+	)
+	(no_connect
+		(at 149.86 133.35)
+	)
+	(no_connect
+		(at 72.39 128.27)
+	)
 	(wire
 		(pts
@@
 	(wire
 		(pts
-			(xy 107.95 148.59) (xy 129.54 148.59)
+			(xy 149.86 143.51) (xy 158.75 143.51)
 		)
 		(stroke
@@
 	(wire
 		(pts
-			(xy 90.17 123.19) (xy 90.17 148.59)
+			(xy 107.95 148.59) (xy 129.54 148.59)
 		)
 		(stroke
@@
 	(wire
 		(pts
-			(xy 149.86 133.35) (xy 158.75 133.35)
+			(xy 90.17 123.19) (xy 90.17 148.59)
 		)
 		(stroke
@@
 	(hierarchical_label "GND"
 		(shape input)
-		(at 153.67 104.14 90)
+		(at 139.7 123.19 90)
 		(effects
 			(font
@@
 		)
 	)
-	(hierarchical_label "GND"
+	(hierarchical_label "SCK"
 		(shape input)
-		(at 139.7 123.19 90)
+		(at 158.75 83.82 0)
 		(effects
 			(font
@@
 		)
 	)
-	(hierarchical_label "SCK"
+	(hierarchical_label "3.3V"
 		(shape input)
-		(at 158.75 83.82 0)
+		(at 139.7 104.14 270)
 		(effects
 			(font
 				(size 1.27 1.27)
 			)
-			(justify left)
+			(justify right)
 		)
 	)
 	(hierarchical_label "3.3V"
 		(shape input)
-		(at 139.7 104.14 270)
+		(at 139.7 157.48 270)
 		(effects
 			(font
@@
 	(hierarchical_label "3.3V"
 		(shape input)
-		(at 139.7 157.48 270)
+		(at 151.13 106.68 270)
 		(effects
 			(font
@@
 		)
 	)
+	(hierarchical_label "GND"
+		(shape input)
+		(at 151.13 101.6 90)
+		(effects
+			(font
+				(size 1.27 1.27)
+			)
+			(justify left)
+		)
+	)
 	(hierarchical_label "MISO"
 		(shape output)
-		(at 158.75 133.35 0)
+		(at 158.75 143.51 0)
 		(effects
 			(font
@@
 		)
 	)
-	(hierarchical_label "3.3V"
-		(shape input)
-		(at 153.67 109.22 270)
-		(effects
-			(font
-				(size 1.27 1.27)
-			)
-			(justify right)
-		)
-	)
 	(symbol
 		(lib_id "Device:R")
@@
 			)
 		)
-		(property "Footprint" "Resistor_SMD:R_0201_0603Metric"
+		(property "Footprint" "Resistor_THT:R_Axial_DIN0207_L6.3mm_D2.5mm_P7.62mm_Horizontal"
 			(at 106.172 144.78 90)
 			(effects
@@
 			)
 		)
-		(property "Footprint" "Capacitor_SMD:C_0201_0603Metric"
+		(property "Footprint" "Capacitor_THT:C_Disc_D5.0mm_W2.5mm_P5.00mm"
 			(at 154.6352 165.1 0)
 			(effects
@@
 	)
 	(symbol
-		(lib_id "PCM_SparkFun-Capacitor:C_Small")
-		(at 153.67 106.68 0)
-		(unit 1)
-		(exclude_from_sim no)
-		(in_bom yes)
-		(on_board yes)
-		(dnp no)
-		(fields_autoplaced yes)
-		(property "Reference" "C20"
-			(at 156.21 102.8762 0)
-			(effects
-				(font
-					(size 1.27 1.27)
-				)
-				(justify left)
-			)
-		)
-		(property "Value" "0.1uF"
-			(at 156.21 105.4162 0)
-			(effects
-				(font
-					(size 1.27 1.27)
-				)
-				(justify left)
-			)
-		)
-		(property "Footprint" "Capacitor_SMD:C_0201_0603Metric"
-			(at 154.6352 118.11 0)
-			(effects
-				(font
-					(size 1.27 1.27)
-				)
-				(hide yes)
-			)
-		)
-		(property "Datasheet" "https://cdn.sparkfun.com/assets/8/a/4/a/5/Kemet_Capacitor_Datasheet.pdf"
-			(at 154.94 123.19 0)
-			(effects
-				(font
-					(size 1.27 1.27)
-				)
-				(hide yes)
-			)
-		)
-		(property "Description" "Unpolarized capacitor"
-			(at 153.67 125.73 0)
-			(effects
-				(font
-					(size 1.27 1.27)
-				)
-				(hide yes)
-			)
-		)
-		(property "PROD_ID" "CAP-00000"
-			(at 153.67 120.65 0)
-			(effects
-				(font
-					(size 1.27 1.27)
-				)
-				(hide yes)
-			)
-		)
-		(property "Voltage" "1kV"
-			(at 156.21 107.9562 0)
-			(effects
-				(font
-					(size 1.27 1.27)
-				)
-				(justify left)
-			)
-		)
-		(property "Tolerance" "100%"
-			(at 156.21 110.4962 0)
-			(effects
-				(font
-					(size 1.27 1.27)
-				)
-				(justify left)
-			)
-		)
-		(pin "1"
-		)
-		(pin "2"
-		)
-		(instances
-			(project "MotherPCB"
-				(path "/ea485091-218e-4ddf-97d6-ebaac999a2f0/11a41087-3c91-483c-9b84-9b4b390ea6bf"
-					(reference "C9")
-					(unit 1)
-				)
-				(path "/ea485091-218e-4ddf-97d6-ebaac999a2f0/27f9d147-2e17-4c91-bb0b-5b3660accb5b"
-					(reference "C3")
-					(unit 1)
-				)
-				(path "/ea485091-218e-4ddf-97d6-ebaac999a2f0/638d8cd3-11c9-4d95-b17c-c3d98881e4a8"
-					(reference "C13")
-					(unit 1)
-				)
-				(path "/ea485091-218e-4ddf-97d6-ebaac999a2f0/ab19c645-77c1-4544-8825-cbc7c98c4ffe"
-					(reference "C17")
-					(unit 1)
-				)
-				(path "/ea485091-218e-4ddf-97d6-ebaac999a2f0/c4c1973d-5436-4e7f-b95e-f77a4f16d85f"
-					(reference "C7")
-					(unit 1)
-				)
-				(path "/ea485091-218e-4ddf-97d6-ebaac999a2f0/d5aabe29-28fd-420f-b684-c56313ee47f3"
-					(reference "C11")
-					(unit 1)
-				)
-				(path "/ea485091-218e-4ddf-97d6-ebaac999a2f0/d8c339b8-6612-4b50-808d-148d2584ca02"
-					(reference "C15")
-					(unit 1)
-				)
-				(path "/ea485091-218e-4ddf-97d6-ebaac999a2f0/da95a8c2-1e5d-4053-8fb4-7b6063b75ac8"
-					(reference "C20")
-					(unit 1)
-				)
-				(path "/ea485091-218e-4ddf-97d6-ebaac999a2f0/f64f5909-243c-44f4-8a0d-0b56181acb9e"
-					(reference "C5")
-					(unit 1)
-				)
-			)
-		)
-	)
-	(symbol
 		(lib_id "Connector:USB3_A")
 		(at 77.47 110.49 0)
@@
 					(unit 1)
 				)
+			)
+		)
+	)
+	(symbol
+		(lib_id "PCM_SparkFun-Capacitor:C_Small")
+		(at 151.13 104.14 0)
+		(unit 1)
+		(exclude_from_sim no)
+		(in_bom yes)
+		(on_board yes)
+		(dnp no)
+		(fields_autoplaced yes)
+		(property "Reference" "C3"
+			(at 153.67 100.3362 0)
+			(effects
+				(font
+					(size 1.27 1.27)
+				)
+				(justify left)
+			)
+		)
+		(property "Value" "0.1uF"
+			(at 153.67 102.8762 0)
+			(effects
+				(font
+					(size 1.27 1.27)
+				)
+				(justify left)
+			)
+		)
+		(property "Footprint" "Capacitor_THT:C_Disc_D5.0mm_W2.5mm_P5.00mm"
+			(at 152.0952 115.57 0)
+			(effects
+				(font
+					(size 1.27 1.27)
+				)
+				(hide yes)
+			)
+		)
+		(property "Datasheet" "https://cdn.sparkfun.com/assets/8/a/4/a/5/Kemet_Capacitor_Datasheet.pdf"
+			(at 152.4 120.65 0)
+			(effects
+				(font
+					(size 1.27 1.27)
+				)
+				(hide yes)
+			)
+		)
+		(property "Description" "Unpolarized capacitor"
+			(at 151.13 123.19 0)
+			(effects
+				(font
+					(size 1.27 1.27)
+				)
+				(hide yes)
+			)
+		)
+		(property "PROD_ID" "CAP-00000"
+			(at 151.13 118.11 0)
+			(effects
+				(font
+					(size 1.27 1.27)
+				)
+				(hide yes)
+			)
+		)
+		(property "Voltage" "1kV"
+			(at 153.67 105.4162 0)
+			(effects
+				(font
+					(size 1.27 1.27)
+				)
+				(justify left)
+			)
+		)
+		(property "Tolerance" "100%"
+			(at 153.67 107.9562 0)
+			(effects
+				(font
+					(size 1.27 1.27)
+				)
+				(justify left)
+			)
+		)
+		(pin "1"
+		)
+		(pin "2"
+		)
+		(instances
+			(project "MotherPCB"
+				(path "/ea485091-218e-4ddf-97d6-ebaac999a2f0/11a41087-3c91-483c-9b84-9b4b390ea6bf"
+					(reference "C11")
+					(unit 1)
+				)
+				(path "/ea485091-218e-4ddf-97d6-ebaac999a2f0/27f9d147-2e17-4c91-bb0b-5b3660accb5b"
+					(reference "C5")
+					(unit 1)
+				)
+				(path "/ea485091-218e-4ddf-97d6-ebaac999a2f0/638d8cd3-11c9-4d95-b17c-c3d98881e4a8"
+					(reference "C15")
+					(unit 1)
+				)
+				(path "/ea485091-218e-4ddf-97d6-ebaac999a2f0/ab19c645-77c1-4544-8825-cbc7c98c4ffe"
+					(reference "C20")
+					(unit 1)
+				)
+				(path "/ea485091-218e-4ddf-97d6-ebaac999a2f0/c4c1973d-5436-4e7f-b95e-f77a4f16d85f"
+					(reference "C9")
+					(unit 1)
+				)
+				(path "/ea485091-218e-4ddf-97d6-ebaac999a2f0/d5aabe29-28fd-420f-b684-c56313ee47f3"
+					(reference "C13")
+					(unit 1)
+				)
+				(path "/ea485091-218e-4ddf-97d6-ebaac999a2f0/d8c339b8-6612-4b50-808d-148d2584ca02"
+					(reference "C17")
+					(unit 1)
+				)
+				(path "/ea485091-218e-4ddf-97d6-ebaac999a2f0/da95a8c2-1e5d-4053-8fb4-7b6063b75ac8"
+					(reference "C3")
+					(unit 1)
+				)
+				(path "/ea485091-218e-4ddf-97d6-ebaac999a2f0/f64f5909-243c-44f4-8a0d-0b56181acb9e"
+					(reference "C7")
+					(unit 1)
+				)
