File: Circuits/MotherPCB/MotherPCB.kicad_pcb (KiCad board)
At the start: 2 copper layers, 144.3 x 122.5 mm, 74 parts, among them J1 USB3_A, J10 USB3_A, J11 USB3_A, J12 USB3_A, J13 USB3_A, J14 USB3_A, J15 USB3_A, J16 Conn_01x03_Pin, J17 Conn_01x06_Socket, J18 USB3_A, J19 Conn_01x06_Socket, J2 PINHD_1x3_Male, J20 Raspberry_Pi_2_3, J21 XT60-M, J3 PINHD_1x3_Male, J4 Conn_01x03_Pin, J5 PINHD_1x5_Male, J8 HX711, J9 USB3_A, U10 MAX3485, U11 MAX3485, U12 MAX3485, U13 MAX3485, U14 MAX3485, U15 MAX3485, U16 MAX3485, U17 MAX3485, U18 ESP32-DEVKITC-32E, U19 MAX3485, U2 MAX3485, U20 Teensy_4.1, U21 MAX3485, U3 MAX3485, U4 MAX3485, U5 MAX3485, U6 MAX3485, U7 MAX3485, U8 MAX3485, U9 MAX3485

Commit message: PCB v2 um
Parts:
- added J6: PINHD_1x3_Male, Connector_PinHeader_2.54mm:PinHeader_1x03_P2.54mm_Vertical, F.Cu at (43.5, 126.6)
- added J7: PINHD_1x3_Male, Connector_PinHeader_2.54mm:PinHeader_1x03_P2.54mm_Vertical, F.Cu at (47.5, 126.6)
- added R12: 10k, Resistor_THT:R_Axial_DIN0207_L6.3mm_D2.5mm_P7.62mm_Horizontal, F.Cu at (51.0, 125.0)
- added R13: 10k, Resistor_THT:R_Axial_DIN0207_L6.3mm_D2.5mm_P7.62mm_Horizontal, F.Cu at (51.1, 128.4)
- added R14: 10k, Resistor_THT:R_Axial_DIN0207_L6.3mm_D2.5mm_P7.62mm_Horizontal, F.Cu at (51.0, 131.9)
Connections:
- J2 pad 1: FLOW_PULSE -> Net-(J2-Pad1)
- J2 pad 3: 3V3 -> Net-(J2-Pad3)
- R20 pad 1: /Tachometer/SIG -> T_PULSE
- R21 pad 2: /Tachometer/SIG -> T_PULSE
- U18 pad J2_19: unconnected-(U18-EXT_5V-PadJ2_19) -> 5V
Routing:
- net T_PULSE: track 0.00 -> 93.9 mm, vias 0 -> 2
- net GND: track 845.4 -> 889.4 mm, vias 11 -> 9
- net SCK_1: track 286.6 -> 312.7 mm, vias 3 -> 7
- net STEPPER_EN: track 102.8 -> 81.2 mm, vias 2 -> 1
- net CS_6: track 133.4 -> 115.8 mm
- net Net-(J2-Pad1): track 0.00 -> 15.2 mm
- net STEPPER_DIR: track 81.4 -> 95.3 mm
- net FLOW_PULSE: track 53.9 -> 67.0 mm
- net Net-(J2-Pad3): track 0.00 -> 12.3 mm
- net CS_5: track 119.1 -> 107.4 mm, vias 1 -> 2
- net /Tachometer/SIG: track 9.36 -> 0.00 mm
- net Net-(R12-Pad2): track 0.00 -> 8.98 mm
- net MOSI_ADC: track 49.3 -> 41.4 mm, vias 1 -> 2
- net CS_3: track 67.7 -> 61.1 mm
- net Net-(J12-SSTX+): track 19.3 -> 14.3 mm
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Other:
- board size 144.3 x 122.5 mm -> 145.2 x 122.5 mm

Commit message: This commit comprises of multiple changes 1. Final MotherPCB (Redesigned by Akshay, only pushed to GitHub by me) 2. PCB for interfacing with the Ethernet MagJack 3. Code for Pressure Transducer data acquisition 4. Inclusion of an ADS1263 Library modified to allow use of SPI1 5. Code for Tachometer re-written as class with static member functions
Parts:
- added J22: PINHD_1x3_Male, Connector_PinHeader_2.54mm:PinHeader_1x03_P2.54mm_Vertical, F.Cu at (149.0, 129.5)
- added J23: Conn_01x08, Connector_PinHeader_2.54mm:PinHeader_1x08_P2.54mm_Vertical, F.Cu at (239.0, 136.3)
- added R15: 10k, Resistor_THT:R_Axial_DIN0207_L6.3mm_D2.5mm_P7.62mm_Horizontal, F.Cu at (149.7, 126.0)
- added R16: 20k, Resistor_THT:R_Axial_DIN0207_L6.3mm_D2.5mm_P7.62mm_Horizontal, F.Cu at (154.0, 130.0)
- moved J21 232.9 mm to (268.2, 104.4), turned to 0 degrees
- moved P1 209.2 mm to (256.2, 95.6), turned to 90 degrees
- moved C7 207.6 mm to (234.2, 123.5)
- moved J18 188.6 mm to (203.7, 127.0), turned to 0 degrees
- moved U19 186.0 mm to (206.7, 117.0), turned to -90 degrees
- moved R10 182.9 mm to (202.5, 119.0), turned to 180 degrees
- moved R21 174.0 mm to (164.0, 22.8), turned to 90 degrees
- moved J1 170.6 mm to (225.2, 127.0), turned to 0 degrees
- moved R20 169.3 mm to (163.8, 26.0), turned to 180 degrees
- moved U21 167.0 mm to (199.2, 113.0), turned to -90 degrees
- moved R2 164.0 mm to (224.0, 119.0), turned to 180 degrees
- moved U4 163.6 mm to (228.2, 117.0), turned to -90 degrees
- moved R9 162.6 mm to (156.0, 22.8), turned to 90 degrees
- moved J4 158.2 mm to (160.0, 22.1), turned to 180 degrees
- moved J5 154.5 mm to (148.0, 16.6), turned to 0 degrees
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Connections:
- J20 pad 11: /PT/DRDY -> DRDY_ADC
- U20 pad 15: unconnected-(U20-A1-Pad15) -> ANLG_2
- U20 pad 16: unconnected-(U20-A2-Pad16) -> ANLG_1
- U20 pad 17: unconnected-(U20-A3-Pad17) -> DRDY_ADC
- U20 pad 20: unconnected-(U20-A6-Pad20) -> Net-(U20-A6)
- U20 pad 28: unconnected-(U20-RX7-Pad28) -> PWM_1
- U20 pad 29: unconnected-(U20-TX7-Pad29) -> PWM_2
- U20 pad 3.3V_1: 3.3V_1 -> 3V3
- U20 pad 3.3V_2: 3.3V -> 3V3
- U20 pad 3.3V_3: 3.3V_2 -> 3V3
- U20 pad 36: unconnected-(U20-CS2-Pad36) -> GPIO_2
- U20 pad 37: unconnected-(U20-CS3-Pad37) -> GPIO
- U20 pad USB_GND1: USB_GND -> USB_GND_1
- U20 pad USB_GND2: USB_GND_1 -> USB_GND
Routing:
- net GND: track 889.4 -> 5.13 mm, vias 9 -> 0
- net 5V: track 252.0 -> 434.7 mm, vias 1 -> 2
- net 3V3: track 599.8 -> 771.2 mm, vias 1 -> 2
- net Net-(U20-A6): track 0.00 -> 118.9 mm, vias 0 -> 2
- net ANLG_2: track 0.00 -> 81.6 mm, vias 0 -> 3
- net PWM_1: track 0.00 -> 81.5 mm, vias 0 -> 1
- net PWM_2: track 0.00 -> 79.8 mm, vias 0 -> 1
- net ANLG_1: track 0.00 -> 79.6 mm, vias 0 -> 3
- net GPIO: track 0.00 -> 74.3 mm, vias 0 -> 1
- net CS_2: track 136.8 -> 66.6 mm
- net CS_5: track 107.4 -> 40.7 mm, vias 2 -> 0
- net GPIO_2: track 0.00 -> 65.2 mm, vias 0 -> 1
- net CS_9: track 142.0 -> 79.0 mm, vias 1 -> 2
- net CS_1: track 36.2 -> 86.9 mm
- net CS_6: track 115.8 -> 69.9 mm
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Other:
- board size 145.2 x 122.5 mm -> 143.5 x 128 mm
- board text added: "3.3V"
- board text added: "3V3"
- board text added: "5V"
- board text added: "ANLG"
- board text added: "DIR"
- board text added: "EN"
- board text added: "GND"
- board text added: "GPIO"
- board text added: "IGN_TGR"
- board text added: "Oil Trigger Modules"
- board text added: "PWM"
- board text added: "Pin 2"
- board text added: "SHRT"
- board text added: "STARTER"
- board text added: "STEPPER"
- board text added: "TACO"
- board text added: "TACOIN"
