File: Circuits/EthernetPCB/EthernetPCB.kicad_sch (KiCad schematic)
At the start: 3 parts, among them J1 Conn_02x03_Counter_Clockwise

Commit message: Final output in thermocouple and ethernet pcb
Verified. Ground plane added. All systems normal.
Connections:
- net GND: now reaches C1.2, J1.4 (Pin_4)
Changed lines of the file:
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@@
 	(text "GND"
 		(exclude_from_sim no)
-		(at 183.134 98.806 0)
+		(at 183.134 97.79 0)
 		(effects
 			(font
@@
 	)
 	(junction
+		(at 186.69 119.38)
+		(diameter 0)
+		(color 0 0 0 0)
+	)
+	(junction
 		(at 66.04 102.87)
 		(diameter 0)
@@
 		(pts
 			(xy 66.04 87.63) (xy 72.39 87.63)
+		)
+		(stroke
+			(width 0)
+			(type default)
+		)
+	)
+	(wire
+		(pts
+			(xy 186.69 119.38) (xy 186.69 128.27)
 		)
 		(stroke
@@
 					(unit 1)
 				)
+			)
+		)
+	)
+	(symbol
+		(lib_id "PCM_SparkFun-PowerSymbol:GND")
+		(at 186.69 128.27 0)
+		(unit 1)
+		(exclude_from_sim no)
+		(in_bom yes)
+		(on_board yes)
+		(dnp no)
+		(fields_autoplaced yes)
+		(property "Reference" "#PWR01"
+			(at 186.69 134.62 0)
+			(effects
+				(font
+					(size 1.27 1.27)
+				)
+				(hide yes)
+			)
+		)
+		(property "Value" "GND"
+			(at 186.69 132.08 0)
+			(do_not_autoplace yes)
+			(effects
+				(font
+					(size 1.27 1.27)
+				)
+			)
+		)
+		(property "Footprint" ""
+			(at 186.69 128.27 0)
+			(effects
+				(font
+					(size 1.27 1.27)
+				)
+				(hide yes)
+			)
+		)
+		(property "Datasheet" ""
+			(at 186.69 128.27 0)
+			(effects
+				(font
+					(size 1.27 1.27)
+				)
+				(hide yes)
+			)
+		)
+		(property "Description" "Power symbol creates a global label with name \"GND\" , ground"
+			(at 186.69 137.16 0)
+			(effects
+				(font
+					(size 1.27 1.27)
+				)
+				(hide yes)
+			)
+		)
+		(pin "1"
+		)
+		(instances
+			(project ""
+				(path "/5162ebe4-85f7-44d0-81d3-1c9d7f16ad6e"
+					(reference "#PWR01")
+					(unit 1)
+				)
