File: Circuits/ThermocouplePCB/ThermocouplePCB.kicad_pcb (KiCad board)
At the start: 2 copper layers, 48 x 21.5 mm, 5 parts, among them J1 USB3_A, J2 Conn_01x06, U1 MAX3485, U2 MAX3485

Commit message: Final output in thermocouple and ethernet pcb
Verified. Ground plane added. All systems normal.
Routing:
- added copper zone on B.Cu, net GND
- added copper zone on F.Cu, net GND
Changed lines of the file:
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@@
 			(outputformat 1)
 			(mirror no)
-			(drillshape 1)
+			(drillshape 0)
 			(scaleselection 1)
-			(outputdirectory "")
+			(outputdirectory "Output/")
 		)
 	)
@@
 		(net 12)
 	)
+	(zone
+		(net 4)
+		(net_name "GND")
+		(layers "F.Cu" "B.Cu")
+		(hatch edge 0.5)
+		(connect_pads
+			(clearance 0.5)
+		)
+		(min_thickness 0.25)
+		(filled_areas_thickness no)
+		(fill yes
+			(thermal_gap 0.5)
+			(thermal_bridge_width 0.5)
+		)
+		(polygon
+			(pts
+				(xy 132.425 91.625) (xy 182.45 91.625) (xy 184.825 94) (xy 184.825 122.525) (xy 182.425 124.925)
+				(xy 134.825 124.925) (xy 126.7 116.8) (xy 126.7 102.5) (xy 126.75 102.45) (xy 126.75 97.3)
+			)
+		)
+	)
 	(embedded_fonts no)
